Commit message: fix joint order

File: Section10_Probability_for_Robotics/bumperbot_ws/src/bumperbot_description/urdf/bumperbot_ros2_control.xacro (robot description, xacro)
@@ -16,5 +16,5 @@
         </xacro:unless>
         <!-- ros2_control Common Interfaces -->
-        <joint name="wheel_right_joint">
+        <joint name="wheel_left_joint">
             <command_interface name="velocity">
               <param name="min">-1</param>
@@ -24,5 +24,5 @@
             <state_interface name="velocity" />
         </joint>
-        <joint name="wheel_left_joint">
+        <joint name="wheel_right_joint">
             <command_interface name="velocity">
               <param name="min">-1</param>

File: Section9_Odometry/bumperbot_ws/src/bumperbot_description/urdf/bumperbot_ros2_control.xacro (robot description, xacro)
@@ -16,5 +16,5 @@
         </xacro:unless>
         <!-- ros2_control Common Interfaces -->
-        <joint name="wheel_right_joint">
+         <joint name="wheel_left_joint">
             <command_interface name="velocity">
               <param name="min">-1</param>
@@ -24,5 +24,5 @@
             <state_interface name="velocity" />
         </joint>
-        <joint name="wheel_left_joint">
+        <joint name="wheel_right_joint">
             <command_interface name="velocity">
               <param name="min">-1</param>
